Commit message: adding gazebo functionality

File: description/robot_core.xacro (robot description, xacro)
@@ -32,4 +32,7 @@
         </xacro:inertial_box>
     </link>
+    <gazebo reference="chassis">
+        <material>Gazebo/White</material>
+    </gazebo>
     <!-- LEFT WHEEL -->
     <joint name="left_wheel_joint" type="continuous">
@@ -55,4 +58,7 @@
         </xacro:inertial_cylinder>
     </link>
+    <gazebo reference="left_wheel">
+        <material>Gazebo/Blue</material>
+    </gazebo>
     <!-- Right WHEEL -->
     <joint name="right_wheel_joint" type="continuous">
@@ -78,4 +84,7 @@
         </xacro:inertial_cylinder>
     </link>
+    <gazebo reference="right_wheel">
+        <material>Gazebo/Blue</material>
+    </gazebo>
     <!-- LEFT CASTER WHEEL -->
     <joint name="left_caster_wheel_joint" type="fixed">
@@ -100,4 +109,9 @@
         </xacro:inertial_sphere>
     </link>
+    <gazebo reference="left_caster_wheel">
+        <material>Gazebo/Black</material>
+        <mu1 value="0.001"/>
+        <mu2 value="0.001"/>
+    </gazebo>
     <!-- RIGHT CASTER WHEEL -->
     <joint name="right_caster_wheel_joint" type="fixed">
@@ -122,3 +136,8 @@
         </xacro:inertial_sphere>
     </link>
+    <gazebo reference="right_caster_wheel">
+        <material>Gazebo/Black</material>
+        <mu1 value="0.001"/>
+        <mu2 value="0.001"/>
+    </gazebo>
 </robot>
