Commit message: before unrolling changes

File: description/gazebo_control.xacro (robot description, xacro)
@@ -2,5 +2,13 @@
 <robot xmlns:xacro="http://www.ros.org/wiki/xacro">
     <gazebo>
-        <plugin name="diff_drive_controller" filename="libgazebo_ros_diff_drive.so">
+        <plugin name="differential_drive_controller" filename="libgazebo_ros_diff_drive.so">
+            <ros>
+                <!-- Set namespace -->
+                <namespace>/</namespace>
+                <!-- Remap default topics -->
+                <argument>--ros-args --remap cmd_vel:=cmd_vel</argument>
+                <argument>--ros-args --remap odom:=odom</argument>
+                <update_rate>10.0</update_rate>
+            </ros>
             <!-- Wheel Information -->
             <left_joint>left_wheel_joint</left_joint>
@@ -12,9 +20,9 @@
             <max_wheel_acceleration>10.0</max_wheel_acceleration>
             <!-- Output -->
-            <odometry_frame>odom</odometry_frame>
-            <robot_base_frame>base_link</robot_base_frame>
             <publish_odom>true</publish_odom>
             <publish_odom_tf>true</publish_odom_tf>
             <publish_wheel_tf>true</publish_wheel_tf>
+            <odometry_frame>odom</odometry_frame>
+            <robot_base_frame>base_link</robot_base_frame>
         </plugin>
     </gazebo>

File: description/robot_core.xacro (robot description, xacro)
@@ -124,5 +124,5 @@
             <geometry>
                 <sphere radius="0.05" />
-            </geometry>
+            </geometry>+++
             <material name="black"/>
         </visual>

Commit message: fixing rviz

File: description/gazebo_control.xacro (robot description, xacro)
@@ -2,13 +2,13 @@
 <robot xmlns:xacro="http://www.ros.org/wiki/xacro">
     <gazebo>
-        <plugin name="differential_drive_controller" filename="libgazebo_ros_diff_drive.so">
-            <ros>
-                <!-- Set namespace -->
-                <namespace>/</namespace>
-                <!-- Remap default topics -->
-                <argument>--ros-args --remap cmd_vel:=cmd_vel</argument>
-                <argument>--ros-args --remap odom:=odom</argument>
-                <update_rate>10.0</update_rate>
-            </ros>
+        <plugin name="gazebo_ros_joint_state_publisher"
+            filename="libgazebo_ros_joint_state_publisher.so">
+            <update_rate>20</update_rate>
+            <joint_name>left_wheel_joint</joint_name>
+            <joint_name>right_wheel_joint</joint_name>
+        </plugin>
+    </gazebo>
+    <gazebo>
+        <plugin name="diff_drive" filename="libgazebo_ros_diff_drive.so">
             <!-- Wheel Information -->
             <left_joint>left_wheel_joint</left_joint>
@@ -20,9 +20,9 @@
             <max_wheel_acceleration>10.0</max_wheel_acceleration>
             <!-- Output -->
+            <odometry_frame>odom</odometry_frame>
+            <robot_base_frame>base_link</robot_base_frame>
             <publish_odom>true</publish_odom>
             <publish_odom_tf>true</publish_odom_tf>
             <publish_wheel_tf>true</publish_wheel_tf>
-            <odometry_frame>odom</odometry_frame>
-            <robot_base_frame>base_link</robot_base_frame>
         </plugin>
     </gazebo>

File: description/robot.urdf.xacro (robot description, xacro)
@@ -1,5 +1,5 @@
 <?xml version="1.0"?>
 <robot xmlns:xacro="http://www.ros.org/wiki/xacro"  name="robot">
-    <xacro:include filename="robot_core.xacro" />
+    <xacro:include filename="tmp_core.xacro" />
     <xacro:include filename="gazebo_control.xacro" />
 </robot>

File: description/robot_core.xacro (robot description, xacro)
@@ -124,5 +124,5 @@
             <geometry>
                 <sphere radius="0.05" />
-            </geometry>+++
+            </geometry>
             <material name="black"/>
         </visual>
